File: EHXSmallClone/SmallClone.sch (KiCad schematic (older format))
At the start: 78 parts, among them J1 Barrel_Jack, Q1 Q_PNP_CBE, Q2 Q_NPN_CBE, Q3 Q_NPN_CBE, Q4 2N7000, SW1 SW_3PDT_on_on, U1 NJM4558, U2 MN3007, U3 4047, U4 LM358

Commit message: schematic update
Connections:
- net 9V: no longer C21.1, C9.2, U2.4 (VGG), U2.5 (VDD)
- net GND: now also C21.1, C9.2, U2.4 (VGG), U2.5 (VDD)
Changed lines of the file:
@@
 LIBS:valves
 LIBS:switches
-LIBS:Untitled-cache
+LIBS:SmallClone-cache
 EELAYER 25 0
 EELAYER END
@@
 $EndComp
 Text Label 14325 2900 2    60   ~ 0
-9V
+GND
 Text Label 12875 2900 0    60   ~ 0
-9V
+GND
 Text Label 10200 1200 3    60   ~ 0
 9V
@@
 $EndComp
 Text Label 12550 1200 3    60   ~ 0
-9V
+GND
 Text Label 15350 5200 2    60   ~ 0
 BBD_CP2
@@
 $EndComp
 Text Label 13025 1200 3    60   ~ 0
-9V
+GND
 Wire Wire Line
 	1825 8675 1900 8675
@@
 	3000 2750 4125 2750
 Wire Wire Line
-	4125 2750 4125 3075
-Wire Wire Line
-	4125 3075 4125 3350
+	4125 2750 4125 3350
 Wire Wire Line
 	3000 2550 3925 2550
@@
 	2300 8575 2625 8575
 Wire Wire Line
-	2925 8575 2975 8575
-Wire Wire Line
-	2975 8575 3050 8575
+	2925 8575 3050 8575
 Wire Wire Line
 	2975 7700 2975 8575
@@
 	3225 9175 3225 9050
 Wire Wire Line
-	3225 9050 3575 9050
-Wire Wire Line
-	3575 9050 3725 9050
+	3225 9050 3725 9050
 Wire Wire Line
 	3575 9175 3575 9050
@@
 	3575 9550 4425 9550
 Wire Wire Line
-	4425 8950 4425 9550
-Wire Wire Line
-	4425 9550 4425 9600
-Wire Wire Line
-	4325 8950 4425 8950
-Wire Wire Line
-	4425 8950 4800 8950
+	4425 8950 4425 9600
+Wire Wire Line
+	4325 8950 4800 8950
 Connection ~ 4425 9550
 Wire Wire Line
 	4425 9900 4425 10100
 Wire Wire Line
-	7425 8525 7900 8525
-Wire Wire Line
-	7900 8525 8075 8525
+	7425 8525 8075 8525
 Wire Wire Line
 	7425 9250 7425 9450
 Wire Wire Line
-	7900 8525 7900 8950
-Wire Wire Line
-	7900 8950 7900 9300
-Wire Wire Line
-	8775 8425 8775 8950
-Wire Wire Line
-	8775 8950 8775 9300
-Wire Wire Line
-	8675 8425 8775 8425
-Wire Wire Line
-	8775 8425 8825 8425
+	7900 8525 7900 9300
+Wire Wire Line
+	8775 8425 8775 9300
+Wire Wire Line
+	8675 8425 8825 8425
 Connection ~ 8775 8425
 Wire Wire Line
 	9125 8425 9175 8425
 Wire Wire Line
-	9475 8425 9550 8425
-Wire Wire Line
-	9550 8425 9700 8425
+	9475 8425 9700 8425
 Wire Wire Line
 	9700 8425 9700 8850
@@
 	4300 6250 4300 6475
 Wire Wire Line
-	4300 5450 5200 5450
-Wire Wire Line
-	5200 5450 5450 5450
+	4300 5450 5450 5450
 Wire Wire Line
 	4300 5450 4300 5500
@@
 	1725 5600 1850 5600
 Wire Wire Line
-	2250 5700 2350 5700
-Wire Wire Line
-	2350 5700 2475 5700
+	2250 5700 2475 5700
 Wire Wire Line
 	1425 5600 1175 5600
 Wire Wire Line
-	2775 5700 2925 5700
-Wire Wire Line
-	2925 5700 3125 5700
+	2775 5700 3125 5700
 Wire Wire Line
 	2925 5825 2925 5700
@@
 	5200 7700 5200 7025
 Wire Wire Line
-	3650 7700 4200 7700
-Wire Wire Line
-	4200 7700 4550 7700
-Wire Wire Line
-	4550 7700 5200 7700
-Wire Wire Line
-	5200 7700 7425 7700
-Wire Wire Line
-	5750 5450 5925 5450
-Wire Wire Line
-	5925 5450 6225 5450
+	3650 7700 7425 7700
+Wire Wire Line
+	5750 5450 6225 5450
 Wire Wire Line
 	5925 5450 5925 5600
@@
 	4200 7700 4200 7775
 Wire Wire Line
-	4550 7500 4550 7700
-Wire Wire Line
-	4550 7700 4550 7775
+	4550 7500 4550 7775
 Connection ~ 4550 7700
 Connection ~ 4200 7700
@@
 	3350 7700 2975 7700
 Wire Wire Line
-	4225 2550 4950 2550
-Wire Wire Line
-	4950 2550 6375 2550
-Wire Wire Line
-	6375 2550 6650 2550
+	4225 2550 6650 2550
 Wire Wire Line
 	6375 2950 6625 2950
 Connection ~ 6375 2950
 Wire Wire Line
-	6375 3300 6375 3350
-Wire Wire Line
-	6375 3350 6375 3400
-Wire Wire Line
-	6375 2450 6375 2550
-Wire Wire Line
-	6375 2550 6375 2600
-Wire Wire Line
-	6375 2900 6375 2950
-Wire Wire Line
-	6375 2950 6375 3000
+	6375 3300 6375 3400
+Wire Wire Line
+	6375 2450 6375 2600
+Wire Wire Line
+	6375 2900 6375 3000
 Connection ~ 6375 2550
 Wire Wire Line
@@
 	10950 1650 10950 1550
 Wire Wire Line
-	10850 1550 10950 1550
-Wire Wire Line
-	10950 1550 11025 1550
+	10850 1550 11025 1550
 Connection ~ 10950 1550
 Wire Wire Line
 	11325 1750 11325 1925
 Wire Wire Line
-	11325 1925 12550 1925
-Wire Wire Line
-	12550 1925 13025 1925
-Wire Wire Line
-	13025 1925 14075 1925
-Wire Wire Line
-	13025 1800 13025 1925
-Wire Wire Line
-	13025 1925 13025 2300
+	11325 1925 14075 1925
+Wire Wire Line
+	13025 1800 13025 2300
 Wire Wire Line
 	14025 2900 14325 2900
@@
 	10200 1550 10550 1550
 Wire Wire Line
-	10200 1200 10200 1550
-Wire Wire Line
-	10200 1550 10200 1800
+	10200 1200 10200 1800
 Connection ~ 10200 1550
 Wire Wire Line
@@
 	10950 1950 10950 2150
 Wire Wire Line
-	9500 1950 9875 1950
-Wire Wire Line
-	9875 1950 10050 1950
+	9500 1950 10050 1950
 Wire Wire Line
 	10725 2700 10725 3225
@@
 	10725 3525 10725 3825
 Wire Wire Line
-	10600 2700 10725 2700
-Wire Wire Line
-	10725 2700 10900 2700
+	10600 2700 10900 2700
 Connection ~ 10725 2700
 Wire Wire Line
-	11200 2700 11300 2700
-Wire Wire Line
-	11300 2700 11400 2700
+	11200 2700 11400 2700
 Wire Wire Line
 	11300 2700 11300 2825
 Wire Wire Line
-	11300 3125 11300 3175
-Wire Wire Line
-	11300 3175 11300 3225
+	11300 3125 11300 3225
 Wire Wire Line
 	11300 3525 11300 3825
 Connection ~ 11300 2700
 Wire Wire Line
-	11700 2700 11800 2700
-Wire Wire Line
-	11800 2700 11900 2700
+	11700 2700 11900 2700
 Wire Wire Line
 	11800 2700 11800 2975
@@
 Connection ~ 11800 2700
 Wire Wire Line
-	6525 5175 6700 5175
-Wire Wire Line
-	6700 5175 7100 5175
+	6525 5175 7100 5175
 Wire Wire Line
 	6700 5175 6700 5400
@@
 	7100 5475 7100 5700
 Wire Wire Line
-	12200 2700 12550 2700
-Wire Wire Line
-	12550 2700 12800 2700
+	12200 2700 12800 2700
 Wire Wire Line
 	12550 2700 12550 2475
@@
 	7550 5975 7550 5750
 Wire Wire Line
-	6225 5975 6700 5975
-Wire Wire Line
-	6700 5975 7550 5975
+	6225 5975 7550 5975
 Wire Wire Line
 	8150 5375 8150 5500
 Wire Wire Line
-	7550 5100 7550 5375
-Wire Wire Line
-	7550 5375 7550 5450
+	7550 5100 7550 5450
 Wire Wire Line
 	14475 2500 14025 2500
@@
 	12925 6200 13025 6200
 Wire Wire Line
-	12925 5800 12925 6000
-Wire Wire Line
-	12925 6000 12925 6200
+	12925 5800 12925 6200
 Wire Wire Line
 	12925 6000 13450 6000
 Wire Wire Line
-	13325 6200 13425 6200
-Wire Wire Line
-	13425 6200 13450 6200
+	13325 6200 13450 6200
 Wire Wire Line
 	13025 5800 12925 5800
@@
 	13175 5600 13450 5600
 Wire Wire Line
-	13175 5200 13175 5400
-Wire Wire Line
-	13175 5400 13175 5600
+	13175 5200 13175 5600
 Wire Wire Line
 	13175 5400 13450 5400
 Wire Wire Line
-	12900 5200 13175 5200
-Wire Wire Line
-	13175 5200 13450 5200
+	12900 5200 13450 5200
 Wire Wire Line
 	13325 5100 13450 5100
 Wire Wire Line
-	13325 4350 13325 4425
-Wire Wire Line
-	13325 4425 13325 4800
-Wire Wire Line
-	13325 4800 13325 4900
-Wire Wire Line
-	13325 4900 13325 5100
+	13325 4350 13325 5100
 Wire Wire Line
 	13325 4800 13450 4800
@@
 Connection ~ 13325 4900
 Wire Wire Line
-	12425 4425 13325 4425
-Wire Wire Line
-	13325 4425 14150 4425
+	12425 4425 14150 4425
 Wire Wire Line
 	14150 4425 14150 4500
@@
 Connection ~ 13425 6200
 Wire Wire Line
-	11000 6550 11200 6550
-Wire Wire Line
-	11200 6550 11525 6550
-Wire Wire Line
-	11525 6550 11800 6550
-Wire Wire Line
-	10275 6550 10450 6550
-Wire Wire Line
-	10450 6550 10700 6550
+	11000 6550 11800 6550
+Wire Wire Line
+	10275 6550 10700 6550
 Wire Wire Line
 	11525 6700 11525 6550
@@
 	11200 7500 11200 7700
 Wire Wire Line
-	10175 5275 10450 5275
-Wire Wire Line
-	10450 5275 10600 5275
+	10175 5275 10600 5275
 Wire Wire Line
 	10450 5275 10450 6550
@@
 	9875 5275 9475 5275
 Wire Wire Line
-	9475 4150 9475 5275
-Wire Wire Line
-	9475 5275 9475 6650
+	9475 4150 9475 6650
 Wire Wire Line
 	9475 6650 9675 6650
@@
 Connection ~ 9475 5275
 Wire Wire Line
-	9850 4300 9850 4375
-Wire Wire Line
-	9850 4375 9850 4475
+	9850 4300 9850 4475
 Wire Wire Line
 	9850 4775 9850 5100
@@
 	11075 4375 11825 4375
 Wire Wire Line
-	11825 4375 11825 4700
-Wire Wire Line
-	11825 4700 11825 5375
+	11825 4375 11825 5375
 Wire Wire Line
 	11825 5375 11700 5375
@@
 	10975 4700 10975 5275
 Wire Wire Line
-	10900 5275 10975 5275
-Wire Wire Line
-	10975 5275 11100 5275
+	10900 5275 11100 5275
 Connection ~ 10975 5275
 Connection ~ 10450 5275
@@
 	9200 1950 8775 1950
 Wire Wire Line
-	12550 1800 12550 1925
-Wire Wire Line
-	12550 1925 12550 2175
+	12550 1800 12550 2175
 Connection ~ 12550 1925
 Wire Wire Line
@@
 Connection ~ 6700 5975
 Wire Wire Line
-	6225 5375 6225 5450
-Wire Wire Line
-	6225 5450 6225 5550
+	6225 5375 6225 5550
 Wire Wire Line
 	6225 5975 6225 5850
